Commit message: merged changes between local versions

File: share/urdf/pepper_awesome.urdf (robot description, URDF)
Before this commit: robot JulietteY20MP, 83 links, 82 joints
Links:
- link Hip: geometry collision mesh filename=package://pepper_description/meshes/HipRoll_0.10.stl scale=0.1 0.1 0.1; visual mesh filename=package://pepper_description/meshes/HipRoll.dae scale=0.1 0.1 0.1
- link Pelvis: geometry collision mesh filename=package://pepper_description/meshes/HipPitch_0.10.stl scale=0.1 0.1 0.1; visual mesh filename=package://pepper_description/meshes/HipPitch.dae scale=0.1 0.1 0.1
- link torso: geometry collision mesh filename=package://pepper_description/meshes/Torso_0.10.stl scale=0.1 0.1 0.1; visual mesh filename=package://pepper_description/meshes/Torso.dae scale=0.1 0.1 0.1
Joints:
- joint HeadYaw: origin xyz=-0.038 0 0.1699 rpy=0 0 0 -> xyz=-0.038 0 0.3089 rpy=0 0 0
- joint HipPitch: axis 0 1.0 0 -> 0 -1.0 0; child Pelvis -> Hip; origin xyz=0 0 -0.079 rpy=0 0 0 -> xyz=0 0 0.268 rpy=0 0 0; parent Hip -> Pelvis
- joint HipRoll: axis 1.0 0 0 -> -1.0 0 0; child Hip -> torso; origin xyz=2e-05 0 -0.139 rpy=0 0 0 -> xyz=0 0 0.079 rpy=0 0 0; parent torso -> Hip
- joint KneePitch: axis 0 1.0 0 -> 0 -1.0 0; child Tibia -> Pelvis; origin xyz=0 0 -0.268 rpy=0 0 0 -> xyz=0 0 0 rpy=0 0 0; parent Pelvis -> Tibia
- joint LShoulderPitch: origin xyz=-0.057 0.14974 0.08682 rpy=0 0 0 -> xyz=-0.057 0.14974 0.22582 rpy=0 0 0
- joint RShoulderPitch: origin xyz=-0.057 -0.14974 0.08682 rpy=0 0 0 -> xyz=-0.057 -0.14974 0.22582 rpy=0 0 0
- joint base_footprint_joint: child base_footprint -> Tibia; origin xyz=0 0 -0.334 rpy=0 0 0 -> xyz=0 0 0.334 rpy=0 0 0; parent Tibia -> base_footprint
- joint base_link_fixedjoint: child torso -> base_link; parent base_link -> torso
